File: experiments/EXP_008/kicad/mycelium_board/_autosave-mycelium_board.kicad_pcb (KiCad board)
At the start: 2 copper layers, 56 parts, among them U1 ?, U10 ?, U11 ?, U12 ?, U13 ?, U14 ?, U15 ?, U16 ?, U17 ?, U18 ?, U19 ?, U2 ?, U20 ?, U21 ?, U22 ?, U23 ?, U24 ?, U25 ?, U26 ?, U27 ?, U28 ?, U29 ?, U3 ?, U30 ?, U31 ?, U32 ?, U33 ?, U34 ?, U35 ?, U36 ?, U37 ?, U38 ?, U39 ?, U4 ?, U40 ?, U41 ?, U42 ?, U43 ?, U44 ?, U45 ?, U46 ?, U47 ?, U48 ?, U49 ?, U5 ?, U50 ?, U51 ?, U52 ?, U53 ?, U54 ?, U55 ?, U56 ?, U6 ?, U7 ?, U8 ?, U9 ?

Commit message: chore: update fab-planner submodule, deploy workflow, and accumulated changes
Parts:
- moved U41 80.1 mm to (143.0, 64.5), turned to -90 degrees
Other:
- board outline added: 80.5 x 90 mm
- copper layers 2 -> 4
Changed lines of the file:
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@@
 	(layers
 		(0 "F.Cu" signal)
+		(1 "In1.Cu" power)
+		(2 "In2.Cu" power)
 		(31 "B.Cu" signal)
 		(32 "B.Adhes" user "B.Adhesive")
@@
 	)
 	(setup
+		(stackup
+			(layer "F.SilkS"
+				(type "Top Silk Screen")
+			)
+			(layer "F.Paste"
+				(type "Top Solder Paste")
+			)
+			(layer "F.Mask"
+				(type "Top Solder Mask")
+				(thickness 0.01)
+			)
+			(layer "F.Cu"
+				(type "copper")
+				(thickness 0.035)
+			)
+			(layer "dielectric 1"
+				(type "prepreg")
+				(thickness 0.1)
+				(material "FR4")
+				(epsilon_r 4.5)
+				(loss_tangent 0.02)
+			)
+			(layer "In1.Cu"
+				(type "copper")
+				(thickness 0.035)
+			)
+			(layer "dielectric 2"
+				(type "core")
+				(thickness 1.24)
+				(material "FR4")
+				(epsilon_r 4.5)
+				(loss_tangent 0.02)
+			)
+			(layer "In2.Cu"
+				(type "copper")
+				(thickness 0.035)
+			)
+			(layer "dielectric 3"
+				(type "prepreg")
+				(thickness 0.1)
+				(material "FR4")
+				(epsilon_r 4.5)
+				(loss_tangent 0.02)
+			)
+			(layer "B.Cu"
+				(type "copper")
+				(thickness 0.035)
+			)
+			(layer "B.Mask"
+				(type "Bottom Solder Mask")
+				(thickness 0.01)
+			)
+			(layer "B.Paste"
+				(type "Bottom Solder Paste")
+			)
+			(layer "B.SilkS"
+				(type "Bottom Silk Screen")
+			)
+			(copper_finish "None")
+			(dielectric_constraints no)
+		)
 		(pad_to_mask_clearance 0)
 		(allow_soldermask_bridges_in_footprints no)
@@
 	(footprint "lib:WIFI-SMD_ESP32-S3-WROOM-1"
 		(layer "F.Cu")
-		(at 80 114 180)
+		(at 143 64.5 -90)
 		(property "Reference" "U41"
-			(at 0 -12 360)
+			(at 0 -12 90)
 			(layer "F.SilkS")
 			(effects
@@
 		)
 		(property "Value" "?"
-			(at 0 12 360)
+			(at 0 12 90)
 			(layer "F.Fab")
 			(effects
@@
 		)
 		(property "Footprint" ""
-			(at 0 0 360)
+			(at 0 0 90)
 			(layer "F.Fab")
 			(hide yes)
@@
 		)
 		(property "Datasheet" ""
-			(at 0 0 360)
+			(at 0 0 90)
 			(layer "F.Fab")
 			(hide yes)
@@
 		)
 		(property "Description" ""
-			(at 0 0 360)
+			(at 0 0 90)
 			(layer "F.Fab")
 			(hide yes)
@@
 		(attr smd)
 		(fp_line
-			(start 9 10.75)
-			(end -9 10.75)
+			(start -9 10.75)
+			(end -9 -10.75)
 			(stroke
 				(width 0.12)
@@
 		)
 		(fp_line
-			(start 9 -10.75)
-			(end 9 10.75)
+			(start 9 10.75)
+			(end -9 10.75)
 			(stroke
 				(width 0.12)
@@
 		)
 		(fp_line
-			(start -9 10.75)
-			(end -9 -10.75)
+			(start -9 -10.75)
+			(end 9 -10.75)
 			(stroke
 				(width 0.12)
@@
 		)
 		(fp_line
-			(start -9 -10.75)
-			(end 9 -10.75)
+			(start 9 -10.75)
+			(end 9 10.75)
 			(stroke
 				(width 0.12)
@@
 		)
 		(pad "1" smd rect
-			(at -8.5 -8.74 180)
+			(at -8.5 -8.74 270)
 			(size 1.8 0.9)
 			(layers "F.Cu" "F.Paste" "F.Mask")
 		)
 		(pad "2" smd rect
-			(at -8.5 -7.47 180)
+			(at -8.5 -7.47 270)
 			(size 1.8 0.9)
 			(layers "F.Cu" "F.Paste" "F.Mask")
@@
 		)
 		(pad "3" smd rect
-			(at -8.5 -6.2 180)
+			(at -8.5 -6.2 270)
 			(size 1.8 0.9)
 			(layers "F.Cu" "F.Paste" "F.Mask")
@@
 		)
 		(pad "4" smd rect
-			(at -8.5 -4.93 180)
+			(at -8.5 -4.93 270)
 			(size 1.8 0.9)
 			(layers "F.Cu" "F.Paste" "F.Mask")
 		)
 		(pad "5" smd rect
-			(at -8.5 -3.66 180)
+			(at -8.5 -3.66 270)
 			(size 1.8 0.9)
 			(layers "F.Cu" "F.Paste" "F.Mask")
@@
 		)
 		(pad "6" smd rect
-			(at -8.5 -2.39 180)
+			(at -8.5 -2.39 270)
 			(size 1.8 0.9)
 			(layers "F.Cu" "F.Paste" "F.Mask")
 		)
 		(pad "7" smd rect
-			(at -8.5 -1.12 180)
+			(at -8.5 -1.12 270)
 			(size 1.8 0.9)
 			(layers "F.Cu" "F.Paste" "F.Mask")
@@
 		)
 		(pad "8" smd rect
-			(at -8.5 0.15 180)
+			(at -8.5 0.15 270)
 			(size 1.8 0.9)
 			(layers "F.Cu" "F.Paste" "F.Mask")
@@
 		)
 		(pad "9" smd rect
-			(at -8.5 1.42 180)
+			(at -8.5 1.42 270)
 			(size 1.8 0.9)
 			(layers "F.Cu" "F.Paste" "F.Mask")
@@
 		)
 		(pad "10" smd rect
-			(at -8.5 2.69 180)
+			(at -8.5 2.69 270)
 			(size 1.8 0.9)
 			(layers "F.Cu" "F.Paste" "F.Mask")
 		)
 		(pad "11" smd rect
-			(at -8.5 3.96 180)
+			(at -8.5 3.96 270)
 			(size 1.8 0.9)
 			(layers "F.Cu" "F.Paste" "F.Mask")
 		)
 		(pad "12" smd rect
-			(at -8.5 5.23 180)
+			(at -8.5 5.23 270)
 			(size 1.8 0.9)
 			(layers "F.Cu" "F.Paste" "F.Mask")
 		)
 		(pad "13" smd rect
-			(at -8.5 6.5 180)
+			(at -8.5 6.5 270)
 			(size 1.8 0.9)
 			(layers "F.Cu" "F.Paste" "F.Mask")
 		)
 		(pad "14" smd rect
-			(at -8.5 7.77 180)
+			(at -8.5 7.77 270)
 			(size 1.8 0.9)
 			(layers "F.Cu" "F.Paste" "F.Mask")
@@
 		)
 		(pad "15" smd rect
-			(at -5.715 10.25 180)
+			(at -5.715 10.25 270)
 			(size 0.9 1.8)
 			(layers "F.Cu" "F.Paste" "F.Mask")
 		)
 		(pad "16" smd rect
-			(at -4.445 10.25 180)
+			(at -4.445 10.25 270)
 			(size 0.9 1.8)
 			(layers "F.Cu" "F.Paste" "F.Mask")
@@
 		)
 		(pad "17" smd rect
-			(at -3.175 10.25 180)
+			(at -3.175 10.25 270)
 			(size 0.9 1.8)
 			(layers "F.Cu" "F.Paste" "F.Mask")
@@
 		)
 		(pad "18" smd rect
-			(at -1.905 10.25 180)
+			(at -1.905 10.25 270)
 			(size 0.9 1.8)
 			(layers "F.Cu" "F.Paste" "F.Mask")
@@
 		)
 		(pad "19" smd rect
-			(at -0.635 10.25 180)
+			(at -0.635 10.25 270)
 			(size 0.9 1.8)
 			(layers "F.Cu" "F.Paste" "F.Mask")
@@
 		)
 		(pad "20" smd rect
-			(at 0.635 10.25 180)
+			(at 0.635 10.25 270)
 			(size 0.9 1.8)
 			(layers "F.Cu" "F.Paste" "F.Mask")
 		)
 		(pad "21" smd rect
-			(at 1.905 10.25 180)
+			(at 1.905 10.25 270)
 			(size 0.9 1.8)
 			(layers "F.Cu" "F.Paste" "F.Mask")
 		)
 		(pad "22" smd rect
-			(at 3.175 10.25 180)
+			(at 3.175 10.25 270)
 			(size 0.9 1.8)
 			(layers "F.Cu" "F.Paste" "F.Mask")
 		)
 		(pad "23" smd rect
-			(at 4.445 10.25 180)
+			(at 4.445 10.25 270)
 			(size 0.9 1.8)
 			(layers "F.Cu" "F.Paste" "F.Mask")
 		)
 		(pad "24" smd rect
-			(at 5.715 10.25 180)
+			(at 5.715 10.25 270)
 			(size 0.9 1.8)
 			(layers "F.Cu" "F.Paste" "F.Mask")
 		)
 		(pad "25" smd rect
-			(at 8.5 7.77 180)
+			(at 8.5 7.77 270)
 			(size 1.8 0.9)
 			(layers "F.Cu" "F.Paste" "F.Mask")
 		)
 		(pad "26" smd rect
-			(at 8.5 6.5 180)
+			(at 8.5 6.5 270)
 			(size 1.8 0.9)
 			(layers "F.Cu" "F.Paste" "F.Mask")
 		)
 		(pad "27" smd rect
-			(at 8.5 5.23 180)
+			(at 8.5 5.23 270)
 			(size 1.8 0.9)
 			(layers "F.Cu" "F.Paste" "F.Mask")
 		)
 		(pad "28" smd rect
-			(at 8.5 3.96 180)
+			(at 8.5 3.96 270)
 			(size 1.8 0.9)
 			(layers "F.Cu" "F.Paste" "F.Mask")
@@
 		)
 		(pad "29" smd rect
-			(at 8.5 2.69 180)
+			(at 8.5 2.69 270)
 			(size 1.8 0.9)
 			(layers "F.Cu" "F.Paste" "F.Mask")
@@
 		)
 		(pad "30" smd rect
-			(at 8.5 1.42 180)
+			(at 8.5 1.42 270)
 			(size 1.8 0.9)
 			(layers "F.Cu" "F.Paste" "F.Mask")
@@
 		)
 		(pad "31" smd rect
-			(at 8.5 0.15 180)
+			(at 8.5 0.15 270)
 			(size 1.8 0.9)
 			(layers "F.Cu" "F.Paste" "F.Mask")
 		)
 		(pad "32" smd rect
-			(at 8.5 -1.12 180)
+			(at 8.5 -1.12 270)
 			(size 1.8 0.9)
 			(layers "F.Cu" "F.Paste" "F.Mask")
 		)
 		(pad "33" smd rect
-			(at 8.5 -2.39 180)
+			(at 8.5 -2.39 270)
 			(size 1.8 0.9)
 			(layers "F.Cu" "F.Paste" "F.Mask")
 		)
 		(pad "34" smd rect
-			(at 8.5 -3.66 180)
+			(at 8.5 -3.66 270)
 			(size 1.8 0.9)
 			(layers "F.Cu" "F.Paste" "F.Mask")
@@
 		)
 		(pad "35" smd rect
-			(at 8.5 -4.93 180)
+			(at 8.5 -4.93 270)
 			(size 1.8 0.9)
 			(layers "F.Cu" "F.Paste" "F.Mask")
@@
 		)
 		(pad "36" smd rect
-			(at 8.5 -6.2 180)
+			(at 8.5 -6.2 270)
 			(size 1.8 0.9)
 			(layers "F.Cu" "F.Paste" "F.Mask")
 		)
 		(pad "37" smd rect
-			(at 8.5 -7.47 180)
+			(at 8.5 -7.47 270)
 			(size 1.8 0.9)
 			(layers "F.Cu" "F.Paste" "F.Mask")
 		)
 		(pad "38" smd rect
-			(at 8.5 -8.74 180)
+			(at 8.5 -8.74 270)
 			(size 1.8 0.9)
 			(layers "F.Cu" "F.Paste" "F.Mask")
@@
 		)
 		(pad "39" smd rect
-			(at 0 -10.25 180)
+			(at 0 -10.25 270)
 			(size 6.7 6.7)
 			(layers "F.Cu" "F.Paste" "F.Mask")
@@
 		)
 		(pad "40" smd rect
-			(at -3.175 -10.25 180)
+			(at -3.175 -10.25 270)
 			(size 0.9 1.8)
 			(layers "F.Cu" "F.Paste" "F.Mask")
 		)
 		(pad "41" smd rect
-			(at 3.175 -10.25 180)
+			(at 3.175 -10.25 270)
 			(size 0.9 1.8)
 			(layers "F.Cu" "F.Paste" "F.Mask")
@@
 		)
 	)
+	(gr_rect
+		(start 64.5 42.5)
+		(end 145 132.5)
+		(stroke
+			(width 0.05)
+			(type default)
+		)
+		(fill none)
+		(layer "Edge.Cuts")
+	)
 )
