File: experiments/EXP_012/pcb/kicad/esp32_motor_controller.kicad_pcb (KiCad board)
At the start: 2 copper layers, 0 parts

Commit message: chore: update fab-planner submodule, deploy workflow, and accumulated changes
Parts:
- added U1: ?, footprints:SOP-8_L4.9-W3.9-P1.27-LS6.0, F.Cu at (115.3, 80.5)
- added U10: ?, footprints:SOT-23-3_L2.9-W1.6-H1.2-LS2.8-BR, F.Cu at (145.4, 84.2)
- added U11: ?, footprints:R0603, F.Cu at (106.4, 69.6)
- added U12: ?, footprints:R0603, F.Cu at (95.9, 101.5)
- added U13: ?, footprints:SOT-23-3_L2.9-W1.6-H1.2-LS2.8-BR, F.Cu at (139.2, 84.2)
- added U14: ?, footprints:R0603, F.Cu at (103.8, 101.3)
- added U15: ?, footprints:R0603, F.Cu at (106.4, 74.1)
- added U16: ?, footprints:SOT-23-3_L2.9-W1.6-H1.2-LS2.8-BR, F.Cu at (132.6, 96.8)
- added U17: ?, footprints:R0603, F.Cu at (103.8, 92.4)
- added U18: ?, footprints:R0603, F.Cu at (141.2, 44.4)
- added U19: ?, footprints:USB-C-SMD_TYPE-C-31-M-12, F.Cu at (95.2, 74.5)
- added U2: ?, footprints:SMA_L4.4-W2.8-LS5.4, F.Cu at (124.2, 100.8)
- added U20: ?, footprints:R0603, F.Cu at (147.1, 39.9)
- added U21: ?, footprints:R0603, F.Cu at (141.2, 48.9)
- added U22: ?, footprints:SOT-23-6_L2.9-W1.6-H1.2-LS2.8-BR, F.Cu at (132.9, 84.2)
- added U23: ?, footprints:SOP-16_L10.0-W3.9-P1.27-LS6.0, F.Cu at (117.5, 70.0)
- added U24: ?, footprints:C0603, F.Cu at (145.8, 100.9)
- added U25: ?, footprints:SOT-23-3_L2.9-W1.6-H1.2-LS2.8-BR, F.Cu at (138.8, 90.5)
- added U26: ?, footprints:SOT-23-3_L2.9-W1.6-H1.2-LS2.8-BR, F.Cu at (145.1, 90.5)
- added U27: ?, footprints:R0603, F.Cu at (95.9, 97.0)
- added U28: ?, footprints:R0603, F.Cu at (89.9, 101.5)
- added U29: ?, footprints:WIFI-SMD_ESP32-WROOM-32, F.Cu at (99.0, 55.9)
- added U3: ?, footprints:IND-SMD_L6.6-W6.6, F.Cu at (140.6, 69.5)
- added U30: ?, footprints:CONN-TH_2P-P5.08_WJ128V-5.0-2P, F.Cu at (131.5, 44.3)
- added U31: ?, footprints:CONN-TH_2P-P5.08_WJ128V-5.0-2P, F.Cu at (117.7, 57.9)
- added U32: ?, footprints:CONN-TH_2P-P5.08_WJ128V-5.0-2P, F.Cu at (94.1, 87.8)
- added U33: ?, footprints:CONN-TH_2P-P5.08_WJ128V-5.0-2P, F.Cu at (117.7, 44.3)
- added U34: ?, footprints:HDR-TH_4P-P2.54-V, F.Cu at (126.2, 78.2)
- added U35: ?, footprints:SW-SMD_L5.1-W5.1-P3.70, F.Cu at (124.5, 85.2)
- added U36: ?, footprints:SW-SMD_L5.1-W5.1-P3.70, F.Cu at (124.5, 93.6)
- added U37: ?, footprints:C0603, F.Cu at (135.9, 77.6)
- added U38: ?, footprints:C0805, F.Cu at (139.2, 101.1)
- added U39: ?, footprints:R0603, F.Cu at (147.1, 44.4)
- added U4: ?, footprints:CAP-SMD_BD6.3-L6.6-W6.6-LS7.6-FD, F.Cu at (144.2, 57.9)
- added U40: ?, footprints:C0603, F.Cu at (148.0, 77.6)
- added U41: ?, footprints:R0603, F.Cu at (103.8, 87.9)
- added U42: ?, footprints:R0603, F.Cu at (106.4, 78.5)
- added U43: ?, footprints:SOD-323_L1.8-W1.3-LS2.5-RD, F.Cu at (132.6, 90.5)
- added U44: ?, footprints:R0603, F.Cu at (147.1, 48.9)
- added U45: ?, footprints:R0603, F.Cu at (103.8, 96.9)
- added U46: ?, footprints:LED0603, F.Cu at (113.6, 92.6)
- added U47: ?, footprints:R0603, F.Cu at (141.2, 39.9)
- added U48: ?, footprints:LED0603, F.Cu at (113.6, 97.3)
- added U49: ?, footprints:R0603, F.Cu at (89.9, 97.0)
- added U5: ?, footprints:CAP-SMD_BD6.3-L6.6-W6.6-LS7.6-FD, F.Cu at (131.0, 57.9)
- added U50: ?, footprints:LED0603, F.Cu at (113.6, 88.0)
- added U51: ?, footprints:R0603, F.Cu at (103.8, 83.5)
- added U6: ?, footprints:C0603, F.Cu at (141.9, 77.6)
- added U7: ?, footprints:SOT-223-3_L6.5-W3.4-H1.6-LS7.0-BR, F.Cu at (129.8, 69.7)
- added U8: ?, footprints:C0805, F.Cu at (139.2, 96.1)
- added U9: ?, footprints:C0805, F.Cu at (146.3, 96.1)
